File: hardware/canary.kicad_pcb (KiCad board)
At the start: 4 copper layers, 100 x 81 mm, 76 parts, among them J102 USB-C 16P, J201 etherCON NE8FBH CAN A, J202 etherCON NE8FBH CAN B, J301 UART/debug 1.27mm, J401 etherCON NE8FBH LAN, SW201 TERMINATE 120R, SW301 RESET, SW302 BOOT, T401 PT61017PEL, U103 AP63200WU, U104 CH224K, U201 ADM3053BRWZ, U301 ESP32-S3-WROOM-1-N8, U401 W5500, Y401 25MHz 10ppm

Commit message: CANary: rename, default name in R1, flush switch cover, insert jig
- Renamed dbCANary -> CANary across docs, firmware, tools, enclosure and the
  KiCad project (files and footprint library nickname). The firmware's NVS
  settings namespace keeps its old name so configured units keep their
  settings; the 0.1.0 changelog entry and board #1's bring-up log and test
  record keep the name they were written under.
- A unit is listed in R1 as "CANary" by default, not the R70 factory "db-70".
- The tube's switch cover sits flush in a 1.2 mm pocket in the lid, with a
  lever notch for a small screwdriver. Not interchangeable with 0.1.0 parts.
- Heat-set insert jig for a common 3D-printed insert press: index plate,
  nest and keyed peg, one socket per insert, verified by posing the real
  tube for every socket.

Co-Authored-By: Claude Opus 5.5 <noreply@anthropic.com>
Parts:
- J201, J202, J401: footprint dbcanary:Neutrik_etherCON_NE8FBH -> canary:Neutrik_etherCON_NE8FBH
Changed lines of the file:
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@@
 		)
 	)
-	(footprint "dbcanary:Neutrik_etherCON_NE8FBH"
+	(footprint "canary:Neutrik_etherCON_NE8FBH"
 		(layer "F.Cu")
 		(at 64 92 180)
@@
 		)
 	)
-	(footprint "dbcanary:Neutrik_etherCON_NE8FBH"
+	(footprint "canary:Neutrik_etherCON_NE8FBH"
 		(layer "F.Cu")
 		(at 36 92 180)
@@
 		)
 	)
-	(footprint "dbcanary:Neutrik_etherCON_NE8FBH"
+	(footprint "canary:Neutrik_etherCON_NE8FBH"
 		(layer "F.Cu")
 		(at 92 92 180)
