File: hardware/ethernet.kicad_sch (KiCad schematic)
At the start: 29 parts, among them J401 etherCON NE8FBH LAN, T401 PT61017PEL, U401 W5500, Y401 25MHz 10ppm

Commit message: CANary: rename, default name in R1, flush switch cover, insert jig
- Renamed dbCANary -> CANary across docs, firmware, tools, enclosure and the
  KiCad project (files and footprint library nickname). The firmware's NVS
  settings namespace keeps its old name so configured units keep their
  settings; the 0.1.0 changelog entry and board #1's bring-up log and test
  record keep the name they were written under.
- A unit is listed in R1 as "CANary" by default, not the R70 factory "db-70".
- The tube's switch cover sits flush in a 1.2 mm pocket in the lid, with a
  lever notch for a small screwdriver. Not interchangeable with 0.1.0 parts.
- Heat-set insert jig for a common 3D-printed insert press: index plate,
  nest and keyed peg, one socket per insert, verified by posing the real
  tube for every socket.

Co-Authored-By: Claude Opus 5.5 <noreply@anthropic.com>
Parts:
- J401: footprint dbcanary:Neutrik_etherCON_NE8FBH -> canary:Neutrik_etherCON_NE8FBH
Changed lines of the file:
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@@
         (font
           (size 1.27 1.27))))
-    (property "Footprint" "dbcanary:Neutrik_etherCON_NE8FBH"
+    (property "Footprint" "canary:Neutrik_etherCON_NE8FBH"
       (at 255.27 85.09 0)
       (effects
